Commit message: Fixed URDF for gazebo

File: robots/edo_gazebo.urdf (robot description, URDF)
Before this commit: robot edo_description, 8 links, 7 joints
Links:
- link link_enf: geometry 
Joints:
- joint joint_1: limit (none) -> lower=-3.1416 upper=3.1416 effort=1000000 velocity=100; type continuous -> revolute
- joint joint_2: limit (none) -> lower=-3.1416 upper=3.1416 effort=1000000 velocity=100; type continuous -> revolute
- joint joint_3: limit (none) -> lower=-3.1416 upper=3.1416 effort=1000000 velocity=100; type continuous -> revolute
- joint joint_4: limit (none) -> lower=-3.1416 upper=3.1416 effort=1000000 velocity=100; type continuous -> revolute
- joint joint_5: limit (none) -> lower=-3.1416 upper=3.1416 effort=1000000 velocity=100; type continuous -> revolute
- joint joint_6: limit (none) -> lower=-3.1416 upper=3.1416 effort=1000000 velocity=100; type continuous -> revolute
- joint joint_7: origin xyz=0 -0.08 0 rpy=0 0 0 -> xyz=0 -0.1136 0 rpy=0 0 0

Commit message: Fix masses and inertia on URDF

File: robots/edo_gazebo.urdf (robot description, URDF)
Before this commit: robot edo_description, 8 links, 7 joints
Links:
- added link world
- link base_link: mass 0.0785942338762368 -> 0.55942338762368
- link link_1: mass 0.0785942338762368 -> 0.55942338762368
- link link_2: mass 0.0785942338762368 -> 0.5
- link link_3: mass 0.0785942338762368 -> 0.5785942338762368
- link link_4: mass 0.0785942338762368 -> 0.5785942338762368
- link link_5: mass 0.0785942338762368 -> 0.5785942338762368
- link link_6: mass 0.0279702497322662 -> 0.5279702497322662
- link link_enf: mass 0.0279702497322662 -> 0.5279702497322662; geometry collision mesh filename=package://edo_description/meshes/cylinder.STL; visual mesh filename=package://edo_description/meshes/cylinder.STL
Joints:
- added joint world_base_joint: type fixed, parent world, child base_link
- joint joint_7: origin xyz=0 -0.1136 0 rpy=0 0 0 -> xyz=0 -0.08 0 rpy=0 0 0
